File: Ingonde_10x10/s_Rangee_1.kicad_sch (KiCad schematic)
At the start: 36 parts, among them J19 Pastille, J20 Pastille, J21 Pastille, J22 Pastille, J23 Pastille, J24 Pastille, J25 Pastille, J26 Pastille, J27 Pastille, J28 Pastille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

Commit message: Ingonde : fin matrice, pastille carrée, vias a 2,54mm
Parts:
- J19, J20, J21, J22, J23, J24, J25, J26, J27, J28, J29, J30, J31, J32, J33, J34, J35, J36, J37, J38, J39, J40, J41, J42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: footprint Chimere_comps:Pastille -> Chimere_comps:Pastille_carree
