File: Ingonde_10x10/s_Rangee_4.kicad_sch (KiCad schematic)
At the start: 36 parts, among them J127 Pastille, J128 Pastille, J129 Pastille, J130 Pastille, J131 Pastille, J132 Pastille, J133 Pastille, J134 Pastille, J135 Pastille, J136 Pastille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

Commit message: Ingonde : fin matrice, pastille carrée, vias a 2,54mm
Parts:
- J127, J128, J129, J130, J131, J132, J133, J134, J135, J136, J137, J138, J139, J140, J141, J142, J143, J144, J145, J146, J147, J148, J149, J150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: footprint Chimere_comps:Pastille -> Chimere_comps:Pastille_carree
