File: Ingonde_10x10/Ingonde_10x10.kicad_sch (KiCad schematic)
At the start: 54 parts, among them J1 2060-451/998-404, J10 2060-451/998-404, J100 Pastille, J101 Pastille, J102 Pastille, J103 Pastille, J104 Pastille, J105 Pastille, J106 Pastille, J107 Pastille, J108 Pastille, J109 Pastille, J11 2060-451/998-404, J110 Pastille, J111 Pastille, J112 Pastille, J113 Pastille, J114 Pastille, J115 Pastille, J116 Pastille, J117 Pastille, J118 Pastille, J119 Pastille, J12 2060-451/998-404, J120 Pastille, J121 Pastille, J122 Pastille, J123 Pastille, J124 Pastille, J125 Pastille, J126 Pastille, J13 2060-451/998-404, J14 2060-451/998-404, J15 2060-451/998-404, J16 2060-451/998-404, J17 2060-451/998-404, J18 2060-451/998-404, J2 2060-451/998-404, J3 2060-451/998-404, J4 2060-451/998-404, J5 2060-451/998-404, J6 2060-451/998-404, J7 2060-451/998-404, J8 2060-451/998-404, J9 2060-451/998-404, J91 Pastille, J92 Pastille, J93 Pastille, J94 Pastille, J95 Pastille, J96 Pastille, J97 Pastille, J98 Pastille, J99 Pastille

Commit message: Ingonde : fin matrice, pastille carrée, vias a 2,54mm
Parts:
- J100, J101, J102, J103, J104, J105, J106, J107, J108, J109, J110, J111, J112, J113, J114, J115, J116, J117, J118, J119, J120, J121, J122, J123, J124, J125, J126, J91, J92, J93, J94, J95, J96, J97, J98, J99: footprint Chimere_comps:Pastille -> Chimere_comps:Pastille_carree
Other:
- added sheet Rangee_21 (s_Rangee_4.kicad_sch)
- added sheet Rangee_22 (s_Rangee_4.kicad_sch)
- added sheet Rangee_23 (s_Rangee_4.kicad_sch)
- added sheet Rangee_24 (s_Rangee_4.kicad_sch)
- added sheet Rangee_25 (s_Rangee_4.kicad_sch)
- added sheet Rangee_26 (s_Rangee_4.kicad_sch)
- added sheet Rangee_27 (s_Rangee_4.kicad_sch)
- added sheet Rangee_28 (s_Rangee_4.kicad_sch)
- added sheet Rangee_29 (s_Rangee_4.kicad_sch)
- added sheet Rangee_30 (s_Rangee_4.kicad_sch)
- added sheet Rangee_31 (s_Rangee_4.kicad_sch)
- added sheet Rangee_32 (s_Rangee_4.kicad_sch)

Commit message: Ingonde_10x10: doublage des connecteurs
Parts:
- J1: footprint Chimere_comps:CONN_2060-1451_998-404_WAGO -> Chimere_comps:Conn_bornier_et_wago
Changed lines of the file:
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@@
 			)
 		)
-		(property "Footprint" "Chimere_comps:CONN_2060-1451_998-404_WAGO"
+		(property "Footprint" "Chimere_comps:Conn_bornier_et_wago"
 			(at 58.42 25.4 0)
 			(effects

Commit message: Ingonde_10x10: fabrication
Parts:
- J10, J11, J12, J13, J14, J15, J16, J17, J18, J2, J3, J4, J5, J6, J7, J8, J9: footprint Chimere_comps:CONN_2060-1451_998-404_WAGO -> Chimere_comps:Conn_bornier_et_wago
Changed lines of the file:
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@@
 			)
 		)
-		(property "Footprint" "Chimere_comps:CONN_2060-1451_998-404_WAGO"
+		(property "Footprint" "Chimere_comps:Conn_bornier_et_wago"
 			(at 223.52 25.4 0)
 			(effects
@@
 			)
 		)
-		(property "Footprint" "Chimere_comps:CONN_2060-1451_998-404_WAGO"
+		(property "Footprint" "Chimere_comps:Conn_bornier_et_wago"
 			(at 83.82 25.4 0)
 			(effects
@@
 			)
 		)
-		(property "Footprint" "Chimere_comps:CONN_2060-1451_998-404_WAGO"
+		(property "Footprint" "Chimere_comps:Conn_bornier_et_wago"
 			(at 261.62 25.4 0)
 			(effects
@@
 			)
 		)
-		(property "Footprint" "Chimere_comps:CONN_2060-1451_998-404_WAGO"
+		(property "Footprint" "Chimere_comps:Conn_bornier_et_wago"
 			(at 274.32 25.4 0)
 			(effects
@@
 			)
 		)
-		(property "Footprint" "Chimere_comps:CONN_2060-1451_998-404_WAGO"
+		(property "Footprint" "Chimere_comps:Conn_bornier_et_wago"
 			(at 185.42 25.4 0)
 			(effects
@@
 			)
 		)
-		(property "Footprint" "Chimere_comps:CONN_2060-1451_998-404_WAGO"
+		(property "Footprint" "Chimere_comps:Conn_bornier_et_wago"
 			(at 96.52 25.4 0)
 			(effects
@@
 			)
 		)
-		(property "Footprint" "Chimere_comps:CONN_2060-1451_998-404_WAGO"
+		(property "Footprint" "Chimere_comps:Conn_bornier_et_wago"
 			(at 172.72 25.4 0)
 			(effects
@@
 			)
 		)
-		(property "Footprint" "Chimere_comps:CONN_2060-1451_998-404_WAGO"
+		(property "Footprint" "Chimere_comps:Conn_bornier_et_wago"
 			(at 248.92 25.4 0)
 			(effects
@@
 			)
 		)
-		(property "Footprint" "Chimere_comps:CONN_2060-1451_998-404_WAGO"
+		(property "Footprint" "Chimere_comps:Conn_bornier_et_wago"
 			(at 134.62 25.4 0)
 			(effects
@@
 			)
 		)
-		(property "Footprint" "Chimere_comps:CONN_2060-1451_998-404_WAGO"
+		(property "Footprint" "Chimere_comps:Conn_bornier_et_wago"
 			(at 210.82 25.4 0)
 			(effects
@@
 			)
 		)
-		(property "Footprint" "Chimere_comps:CONN_2060-1451_998-404_WAGO"
+		(property "Footprint" "Chimere_comps:Conn_bornier_et_wago"
 			(at 160.02 25.4 0)
 			(effects
@@
 			)
 		)
-		(property "Footprint" "Chimere_comps:CONN_2060-1451_998-404_WAGO"
+		(property "Footprint" "Chimere_comps:Conn_bornier_et_wago"
 			(at 198.12 25.4 0)
 			(effects
@@
 			)
 		)
-		(property "Footprint" "Chimere_comps:CONN_2060-1451_998-404_WAGO"
+		(property "Footprint" "Chimere_comps:Conn_bornier_et_wago"
 			(at 147.32 25.4 0)
 			(effects
@@
 			)
 		)
-		(property "Footprint" "Chimere_comps:CONN_2060-1451_998-404_WAGO"
+		(property "Footprint" "Chimere_comps:Conn_bornier_et_wago"
 			(at 109.22 25.4 0)
 			(effects
@@
 			)
 		)
-		(property "Footprint" "Chimere_comps:CONN_2060-1451_998-404_WAGO"
+		(property "Footprint" "Chimere_comps:Conn_bornier_et_wago"
 			(at 121.92 25.4 0)
 			(effects
@@
 			)
 		)
-		(property "Footprint" "Chimere_comps:CONN_2060-1451_998-404_WAGO"
+		(property "Footprint" "Chimere_comps:Conn_bornier_et_wago"
 			(at 71.12 25.4 0)
 			(effects
@@
 			)
 		)
-		(property "Footprint" "Chimere_comps:CONN_2060-1451_998-404_WAGO"
+		(property "Footprint" "Chimere_comps:Conn_bornier_et_wago"
 			(at 236.22 25.4 0)
 			(effects
