File: Basine_10x10/Basine.kicad_pcb (KiCad board)
At the start: 2 copper layers, 100 x 100 mm, 226 parts, among them J1 2060-451/998-404, J10 2060-451/998-404, J100 Pastille, J101 Pastille, J102 Pastille, J103 Pastille, J104 Pastille, J105 Pastille, J106 Pastille, J107 Pastille, J108 Pastille, J109 Pastille, J11 2060-451/998-404, J110 Pastille, J111 Pastille, J112 Pastille, J113 Pastille, J114 Pastille, J115 Pastille, J116 Pastille, J117 Pastille, J118 Pastille, J119 Pastille, J12 2060-451/998-404, J120 Pastille, J121 Pastille, J122 Pastille, J123 Pastille, J124 Pastille, J125 Pastille, J126 Pastille, J127 Pastille, J128 Pastille, J129 Pastille, J13 2060-451/998-404, J130 Pastille, J131 Pastille, J132 Pastille, J133 Pastille, J134 Pastille, J135 Pastille, J136 Pastille, J137 Pastille, J138 Pastille, J139 Pastille, J14 2060-451/998-404, J140 Pastille, J141 Pastille, J142 Pastille, J143 Pastille, J144 Pastille, J145 Pastille, J146 Pastille, J147 Pastille, J148 Pastille, J149 Pastille, J15 2060-451/998-404, J150 Pastille, J151 Pastille, J152 Pastille, J153 Pastille, J154 Pastille, J155 Pastille, J156 Pastille, J157 Pastille, J158 Pastille, J159 Pastille, J16 2060-451/998-404, J160 Pastille, J161 Pastille, J162 Pastille, J163 Pastille, J164 Pastille, J165 Pastille, J166 Pastille, J167 Pastille, J168 Pastille, J169 Pastille, J17 2060-451/998-404, J170 Pastille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

Commit message: maj ultrogothe et fabrication
Other:
- board text added: "A0"
- board text added: "A1"
- board text added: "A2"
- board text added: "A3"
- board text added: "A4"
- board text added: "A5"
- board text added: "A6"
- board text added: "A7"
- board text added: "B1"
- board text added: "B10"
- board text added: "B11"
- board text added: "B12"
- board text added: "B13"
- board text added: "B14"
- board text added: "B15"
- board text added: "B2"
- board text added: "B8"
- board text added: "B9"
